Commit message: final working with training and metrics fixed

File: install/drone_rl/share/drone_rl/urdf/drone_simple.urdf (robot description, URDF)
Before this commit: robot drone, 5 links, 4 joints
Links:
- added link base_footprint
Joints:
- added joint base_joint: type fixed, parent base_footprint, child base_link, origin xyz=0 0 0.1 rpy=0 0 0
- joint lidar_joint: origin xyz=0 0 0.08 rpy=0 0 0 -> xyz=0 0 0.15 rpy=0 0 0

File: src/drone_rl/urdf/drone_simple.urdf (robot description, URDF)
Before this commit: robot drone, 5 links, 4 joints
Links:
- added link base_footprint
Joints:
- added joint base_joint: type fixed, parent base_footprint, child base_link, origin xyz=0 0 0.1 rpy=0 0 0
- joint lidar_joint: origin xyz=0 0 0.08 rpy=0 0 0 -> xyz=0 0 0.15 rpy=0 0 0
